File: aeolus.kicad_pcb (KiCad board)
At the start: 2 copper layers, 80 x 25 mm, 26 parts, among them J1 Barrel_Jack_Switch, J2 Conn_01x04_Pin, Q1 2N3904, U1 XIAO-ESP32-C6-SMD, U2 MPM3610GQV-P, U3 LM66100DCK, U4 EMC2101-ACZL-TR, U5 INA219BIDCNR

Commit message: More progress on PCB
Parts:
- added C8: 0.1u, Capacitor_SMD:C_0805_2012Metric, F.Cu at (101.0, 85.0)
- added C9: 0.1u, Capacitor_SMD:C_0805_2012Metric, F.Cu at (101.0, 88.0)
- added D2: LED, LED_SMD:LED_1206_3216Metric, F.Cu at (91.6, 85.2)
- added D3: LED, LED_SMD:LED_1206_3216Metric, F.Cu at (91.6, 88.6)
- added D4: LED, LED_SMD:LED_1206_3216Metric, F.Cu at (91.6, 92.0)
- added R10: 10k, Resistor_SMD:R_0805_2012Metric, F.Cu at (96.6, 85.0)
- added R11: 10k, Resistor_SMD:R_0805_2012Metric, F.Cu at (96.6, 87.9)
- added R12: 10k, Resistor_SMD:R_0805_2012Metric, F.Cu at (96.6, 90.9)
- added TP1: 12V TP, TestPoint:TestPoint_Pad_D2.0mm, F.Cu at (90.8, 77.4)
- added TP2: 5V TP, TestPoint:TestPoint_Pad_D2.0mm, F.Cu at (90.8, 81.5)
- added TP3: VMCU TP, TestPoint:TestPoint_Pad_D2.0mm, F.Cu at (94.8, 77.4)
- added TP4: 3V3 TP, TestPoint:TestPoint_Pad_D2.0mm, F.Cu at (94.8, 81.5)
- added TP5: SCL, TestPoint:TestPoint_Pad_D2.0mm, F.Cu at (98.9, 77.4)
- added TP6: SDA, TestPoint:TestPoint_Pad_D2.0mm, F.Cu at (98.9, 81.5)
- added TP7: FAN, TestPoint:TestPoint_Pad_D2.0mm, F.Cu at (102.9, 77.4)
- added TP8: TACH, TestPoint:TestPoint_Pad_D2.0mm, F.Cu at (102.9, 81.5)
- R1, R2, R3, R4, R5, R6, R7, R8: footprint Resistor_SMD:R_0201_0603Metric -> Resistor_SMD:R_0805_2012Metric
- moved C4 65.2 mm to (176.0, 81.5)
- moved C5 65.2 mm to (175.8, 72.7)
- moved R5 65.2 mm to (173.7, 81.5)
- moved C3 65.2 mm to (173.1, 76.3)
- moved R7 58.6 mm to (187.9, 91.0), turned to 180 degrees
- moved R6 58.2 mm to (188.0, 96.0), turned to 180 degrees
- moved J1 55.3 mm to (117.0, 106.3)
- moved U1 48.3 mm to (174.5, 97.5)
- moved D1 38.8 mm to (124.5, 96.5)
- moved F1 33.3 mm to (127.9, 104.5), turned to 0 degrees
- moved R9 31.9 mm to (131.9, 95.7)
- moved U3 31.5 mm to (142.3, 92.4), turned to 90 degrees
- moved U5 26.1 mm to (134.4, 75.7)
- moved C7 22.7 mm to (156.2, 62.6)
- moved U4 22.4 mm to (159.6, 97.1), turned to 90 degrees
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Connections:
- net Net-(D1-A2) renamed /DC_IN
- net Net-(U5-VIN+) renamed /VSense+
- net Net-(U5-VIN-) renamed /VSense-
Routing:
- net VDC: track 10.4 -> 0.00 mm
- net +5V: track 0.00 -> 9.60 mm, vias 0 -> 2
- net Net-(U2-FB): track 0.00 -> 7.50 mm
- net +12V: track 15.5 -> 9.16 mm
- net GND: track 10.4 -> 16.4 mm, vias 0 -> 16
- net Net-(U2-EN): track 0.00 -> 4.65 mm
- net Net-(U2-AAM): track 0.00 -> 2.61 mm
- added copper zone on F.Cu, net +12V
- added copper zone on F.Cu, net +5V
- added copper zone on F.Cu, net /DC_IN
- added copper zone on F.Cu, net /SW
- added copper zone on F.Cu, net GND

Commit message: Inital pass at PCB
Parts:
- added C10: 0.1u, Capacitor_SMD:C_0805_2012Metric, F.Cu at (187.7, 99.7)
- added C11: 10u, Capacitor_SMD:C_0805_2012Metric, F.Cu at (190.2, 99.7)
- added C12: 1u, Capacitor_SMD:C_0805_2012Metric_Pad1.18x1.45mm_HandSolder, F.Cu at (151.4, 91.5)
- added H1: MountingHole_Pad, MountingHole:MountingHole_3.2mm_M3_Pad_Via, F.Cu at (125.2, 88.6)
- added H2: MountingHole_Pad, MountingHole:MountingHole_3.2mm_M3_Pad_Via, F.Cu at (197.3, 104.5)
- added J3: Conn_01x04_Pin, Connector:FanPinHeader_1x04_P2.54mm_Vertical, F.Cu at (188.9, 88.7)
- added J4: Conn_01x04_Pin, Connector:FanPinHeader_1x04_P2.54mm_Vertical, F.Cu at (205.9, 88.7)
- added JP1: INA219_A0, Jumper:SolderJumper-2_P1.3mm_Open_TrianglePad1.0x1.5mm, B.Cu at (162.8, 97.8)
- added JP2: INA219_A1, Jumper:SolderJumper-2_P1.3mm_Open_TrianglePad1.0x1.5mm, B.Cu at (165.4, 97.8)
- added R13: 10k, Resistor_SMD:R_0805_2012Metric, F.Cu at (165.4, 94.2)
- added R14: 10k, Resistor_SMD:R_0805_2012Metric, F.Cu at (162.8, 94.2)
- added R15: 0, Resistor_SMD:R_0805_2012Metric_Pad1.20x1.40mm_HandSolder, F.Cu at (148.4, 90.4)
- added R16: 0, Resistor_SMD:R_0805_2012Metric_Pad1.20x1.40mm_HandSolder, F.Cu at (148.4, 92.5)
- added TP10: TACH2, TestPoint:TestPoint_Pad_D2.0mm, B.Cu at (193.4, 90.8)
- added TP9: TACH3, TestPoint:TestPoint_Pad_D2.0mm, B.Cu at (210.8, 90.8)
- added U6: 74LVC3G07, Package_SO:SSOP-8_2.95x2.8mm_P0.65mm, F.Cu at (184.8, 97.9)
- TP3, TP7, TP8: moved to B.Cu
- U1: footprint OPL_Kicad_Library:XIAO-ESP32C6-SMD -> Aeolus:XIAO-ESP32C6-SMD
- U5: value INA219BIDCNR -> INA219BIDR; footprint Package_TO_SOT_SMD:SOT-23-8 -> Package_SO:SOIC-8_3.9x4.9mm_P1.27mm
- moved TP6 139.4 mm to (237.2, 98.5), turned to 180 degrees
- moved TP5 138.0 mm to (236.5, 87.8)
- moved TP3 119.3 mm to (210.7, 105.9), turned to 180 degrees
- moved TP4 117.9 mm to (211.8, 95.9)
- moved D4 113.6 mm to (204.3, 106.0), turned to 90 degrees
- moved R12 108.3 mm to (204.3, 101.6), turned to -90 degrees
- moved D3 79.0 mm to (168.7, 105.9), turned to 90 degrees
- moved C8 74.3 mm to (173.2, 102.9), turned to -90 degrees
- moved TP8 74.3 mm to (176.7, 90.8), turned to 180 degrees
- moved D2 73.7 mm to (162.3, 105.9), turned to 90 degrees
- moved R11 70.8 mm to (165.6, 103.6)
- moved TP7 70.2 mm to (169.5, 99.7), turned to 180 degrees
- moved U3 69.0 mm to (210.3, 104.0), turned to -90 degrees
- moved TP2 67.7 mm to (154.9, 103.1)
- moved R10 65.3 mm to (159.0, 104.4)
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Connections:
- net TACH renamed TACH1
- J2 pad 4: FAN -> FAN1
- U1 pad 10: unconnected-(U1-GPIO20_D9_MISO-Pad10) -> TACH2
- U1 pad 9: unconnected-(U1-GPIO19_D8_SCK-Pad9) -> TACH3
- U5 pad 1: /VSense+ -> Net-(U5-VIN+)
- U5 pad 2: /VSense- -> Net-(U5-VIN-)
- U5 pad 7: GND -> Net-(JP1-A)
- U5 pad 8: GND -> Net-(JP2-A)
Routing:
- net VDC: track 0.00 -> 152.6 mm, vias 0 -> 36
- net +3V3: track 0.00 -> 142.9 mm, vias 0 -> 5
- net SDA: track 0.00 -> 90.3 mm, vias 0 -> 2
- net SCL: track 0.00 -> 89.3 mm, vias 0 -> 2
- net +5V: track 9.60 -> 94.1 mm, vias 2 -> 4
- net TACH2: track 0.00 -> 38.7 mm, vias 0 -> 1
- net +12V: track 9.16 -> 39.1 mm, vias 0 -> 2
- net FAN: track 0.00 -> 25.7 mm, vias 0 -> 1
- net FAN1: track 0.00 -> 25.0 mm, vias 0 -> 1
- net FAN3: track 0.00 -> 22.5 mm, vias 0 -> 2
- net TACH3: track 0.00 -> 21.1 mm, vias 0 -> 1
- net TACH1: track 0.00 -> 18.3 mm, vias 0 -> 1
- net GND: track 16.4 -> 34.6 mm, vias 16 -> 75
- net VCC: track 0.00 -> 15.4 mm, vias 0 -> 2
- net Net-(JP2-A): track 0.00 -> 14.5 mm, vias 0 -> 1
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- added copper zone on F.Cu, net VCC
- added copper zone on B.Cu, net VDC
- added copper zone on F.Cu, net VDC
Other:
- board size 80 x 25 mm -> 120 x 25 mm

Commit message: Migrate to 4 layer board and beef up fan power distribution
Parts:
- added REF**: OSHW-Logo2_7.3x6mm_SilkScreen, Symbol:OSHW-Logo2_7.3x6mm_SilkScreen, F.Cu at (198.0, 97.4)
- added REF**: LayerMarker_4_6.35x2.54mm_TextH1mm_P1.27mm_LowerMirrored, Symbol:LayerMarker_4_6.35x2.54mm_TextH1mm_P1.27mm_LowerMirrored, F.Cu at (188.0, 108.1)
- added REF**: OSHW-Logo2_7.3x6mm_SilkScreen, Symbol:OSHW-Logo2_7.3x6mm_SilkScreen, B.Cu at (230.4, 105.1)
- moved D1 4.67 mm to (137.6, 99.4), turned to 0 degrees
- moved TP4 3.49 mm to (208.4, 96.1)
Connections:
- D1 pad 2: /DC_IN -> +12V
Routing:
- net +3V3: track 142.9 -> 34.8 mm, vias 5 -> 16
- net VDC: track 152.6 -> 218.5 mm
- net GND: track 34.6 -> 43.7 mm, vias 75 -> 74
- net +5V: track 94.1 -> 86.8 mm, vias 4 -> 6
- net +12V: track 39.1 -> 33.5 mm, vias 2 -> 4
- net VCC: track 15.4 -> 19.3 mm
- net Net-(JP2-A): track 14.5 -> 13.6 mm
- net FAN3: track 22.5 -> 21.7 mm
- net Net-(U2-FB): track 7.50 -> 8.07 mm
- added copper zone on F.Cu, net +3V3
- added copper zone on In1.Cu, net +3V3
- added copper zone on In2.Cu, net GND
- added copper zone on In1.Cu, net VDC
- added copper zone on In2.Cu, net VDC
- removed copper zone on B.Cu, net GND
Other:
- copper layers 2 -> 4
